File: teensy_relay_controller.brd (EAGLE design)
At the start: 44.1 x 41.9 mm, 7 parts

Commit message: Cleaning up the size of the board abit
Other:
- board size 44.1 x 41.9 mm -> 44.5 x 44.4 mm
Changed lines of the file:
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@@
 <board>
 <plain>
-<wire x1="0" y1="38.1" x2="44.12" y2="38.1" width="0" layer="20"/>
-<wire x1="44.12" y1="80" x2="0" y2="80" width="0" layer="20"/>
-<wire x1="0" y1="80" x2="0" y2="38.1" width="0" layer="20"/>
+<wire x1="0" y1="38.1" x2="44.45" y2="38.1" width="0" layer="20"/>
+<wire x1="0" y1="82.55" x2="0" y2="38.1" width="0" layer="20"/>
+<wire x1="44.45" y1="82.55" x2="44.45" y2="38.1" width="0" layer="20"/>
+<wire x1="44.45" y1="82.55" x2="0" y2="82.55" width="0" layer="20"/>
 </plain>
 <attributes>
